File: vault35_alpha-rounded.kicad_pcb (KiCad board)
At the start: 2 copper layers, 209.7 x 76.4 mm, 123 parts, among them J1 AVR-ISP-6, SW1 SW_PUSH, SW2 RotaryEncoder_Switch, SW3 RotaryEncoder_Switch, SW5 SW_PUSH, SW6 SW_PUSH, U1 SRV05-4, U2 ATmega32U4-M, X1 Crystal_GND24_Small

Commit message: production
Routing:
- net GND: track 93.4 -> 88.8 mm
- net col5: track 135.4 -> 131.6 mm
- net RST: track 66.2 -> 63.1 mm
- net col8: track 227.6 -> 224.7 mm
- net Net-(C1-Pad1): track 10.1 -> 7.59 mm
- net Net-(UR3-Pad1): track 14.5 -> 12.8 mm
- net SDA: track 83.0 -> 81.4 mm
- net D+: track 37.0 -> 35.5 mm
- net col1: track 59.2 -> 57.7 mm
- net row0: track 228.1 -> 226.6 mm
- net D-: track 39.1 -> 37.7 mm
- net col3: track 123.8 -> 122.4 mm
- net PD5: track 116.4 -> 115.0 mm
- net row3: track 206.7 -> 205.3 mm
- net SCL: track 88.3 -> 86.9 mm
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